Commit message: Update robot_core.xacro wheel radius

File: description/robot_core.xacro (robot description, xacro)
@@ -6,5 +6,5 @@
     <xacro:property name="chassis_height" value="0.145"/>
     <xacro:property name="chassis_mass" value="1.0"/>
-    <xacro:property name="wheel_radius" value="0.286"/>
+    <xacro:property name="wheel_radius" value="0.0286"/>
     <xacro:property name="wheel_thickness" value="0.05"/>
     <xacro:property name="wheel_mass" value="0.05"/>

Commit message: a

File: description/robot_core.xacro (robot description, xacro)
@@ -5,8 +5,8 @@
     <xacro:property name="chassis_width" value="0.156"/>
     <xacro:property name="chassis_height" value="0.145"/>
-    <xacro:property name="chassis_mass" value="1.0"/>
+    <xacro:property name="chassis_mass" value="0.905"/>
     <xacro:property name="wheel_radius" value="0.0286"/>
     <xacro:property name="wheel_thickness" value="0.05"/>
-    <xacro:property name="wheel_mass" value="0.05"/>
+    <xacro:property name="wheel_mass" value="0.02"/>
     <xacro:property name="wheel_offset_x" value="0.018"/>
     <xacro:property name="wheel_offset_y" value="0.078"/>
